Commit message: added floor model and background model for the gazebo visualization

File: urdf/camera.xacro (robot description, xacro)
@@ -84,4 +84,7 @@
       </sensor>
     </gazebo>
+  <gazebo reference="${camera_frame}">
+    <material>Gazebo/Black</material>
+  </gazebo>
   </xacro:macro>
 </robot>
